File: DAPlink_CC.kicad_sch (KiCad schematic)
At the start: 8 parts

Commit message: Update DAPlink_CC.kicad_sch
Parts:
- removed J?: USB_TypeC-16, 206_CONN_USB:HC-16_7426ST, symbol 306_Link_USB-Connector:USB_TypeC-16
- removed R?: 1k, 001_GN_RCL_SMD:R0402(1005M), symbol 001_Basic_PassiveComponents:001_Resistor
- added C? (x2): 100nF, 001_GN_RCL_SMD:C0402(1005M), symbol 001_Basic_PassiveComponents:101_Capacitor
- added J? (x2): USB_TypeC-24, symbol 306_Link_USB-Connector:USB_TypeC-24
- added R? (x2): 100k, 001_GN_RCL_SMD:R0402(1005M), symbol 001_Basic_PassiveComponents:001_Resistor
- added R?: 5.1k, 001_GN_RCL_SMD:R0402(1005M), symbol 001_Basic_PassiveComponents:001_Resistor
- added U?: SL2.1S, 004_GN_MIDDLE-SEMI_SMD:MSOP-16_2646, symbol 110_IntegratedCircuit_Interface:SL2.1S
- added X?: 002_Xtal-4, 006_GN_XTAL_OSC_SMD:CXO-4_3225, symbol 003_Basic_CrystalAndOscillator:002_Xtal-4
Connections:
- net +3V3: now also C?.1, C?.1
- net DAP_CLK: now also J?.A2 (Tx1_P), J?.A8 (SBU1), J?.B2 (Tx2_P)
- net DAP_DIO: now also J?.A3 (Tx1_N), J?.B3 (Tx2_N), J?.B8 (SBU2)
- net DAP_Rx: now also J?.A11 (Rx2_P), J?.B11 (Rx1_P), J?.B5 (CC2)
- net DAP_Tx: now also J?.A10 (Rx2_N), J?.A5 (CC1), J?.B10 (Rx1_N), R?.1
- net DN: now also J?.A7 (DM1), J?.B7 (DM2); no longer U?.19 (PA11)
- net DP: now also J?.A6 (DP1), J?.B6 (DP2); no longer U?.20 (PA12)
- net GND: now also C?.2, C?.2, J?.A1 (GND), J?.A1 (GND), J?.A12 (GND), J?.A12 (GND), J?.B1 (GND), J?.B1 (GND), J?.B12 (GND), J?.B12 (GND), J?.SHELL, J?.SHELL, R?.2
- net UART-Rx: now also J?.A11 (Rx2_P), J?.B11 (Rx1_P)
- net UART-Tx: now also J?.A10 (Rx2_N), J?.B10 (Rx1_N)
- net VDC: now also J?.A4 (VBUS), J?.A9 (VBUS), J?.B4 (VBUS), J?.B9 (VBUS), R?.1, R?.1
- net SWCLK_TCK renamed SWCLK
- net SWCLK: now also J?.A2 (Tx1_P), J?.B2 (Tx2_P)
- net SWDIO_TMS renamed SWDIO
- net SWDIO: now also J?.A3 (Tx1_N), J?.B3 (Tx2_N)
- new net DAP_DN: U?.19 (PA11)
- new net DAP_DP: U?.20 (PA12)
- new net DVC-DN: J?.A7 (DM1), J?.B7 (DM2)
- new net DVC-DP: J?.A6 (DP1), J?.B6 (DP2)
- new net SWD-SBU1: J?.A8 (SBU1)
- new net SWD-SBU2: J?.B8 (SBU2)
- new net UART-CC1: J?.A5 (CC1), R?.2
- new net UART-CC2: J?.B5 (CC2), R?.2
- new net VBUS: J?.A4 (VBUS), J?.A9 (VBUS), J?.B4 (VBUS), J?.B9 (VBUS)
- no-connect marks 12 -> 10
Other:
- moved on the sheet: U?C

Commit message: Update DAPlink_CC.kicad_sch
Parts:
- removed U?: SL2.1S, 004_GN_MIDDLE-SEMI_SMD:MSOP-16_2646, symbol 110_IntegratedCircuit_Interface:SL2.1S
- added C? (x3): 100nF, 001_GN_RCL_SMD:C0402(1005M), symbol 001_Basic_PassiveComponents:101_Capacitor
- added C? (x2): 10pF, 001_GN_RCL_SMD:C0402(1005M), symbol 001_Basic_PassiveComponents:101_Capacitor
- added U?: SL2.1S, 004_GN_MIDDLE-SEMI_SMD:MSOP-16_2646, symbol 110_IntegratedCircuit_Interface:SL2.1S
Connections:
- net DAP_DN: now also U?.3 (DM1)
- net DAP_DP: now also U?.4 (DP1)
- net DN: now also U?.5 (DM_U)
- net DP: now also U?.6 (DP_U)
- net DVC-DN: now also U?.1 (DM2)
- net DVC-DP: now also U?.2 (DP2)
- net GND: now also X?.2, X?.4, C?.1, C?.1, C?.2, C?.2, C?.2, U?.8 (GND)
- net VBUS: now also C?.1, U?.7 (Vin_5V)
- net at X?.1: now also C?.2, U?.12 (XTAL_IN)
- net at X?.3: now also C?.2, U?.11 (XTAL_OUT)
- new net: C?.1, U?.10 (V_1V8)
- new net: C?.1, U?.9 (V_3V3)
- no-connect marks 10 -> 14
Other:
- moved on the sheet: X?

Commit message: Update DAPlink_CC.kicad_sch
Parts:
- removed C? (x5): 100nF, 001_GN_RCL_SMD:C0402(1005M), symbol 001_Basic_PassiveComponents:101_Capacitor
- removed C?: 10pF, 001_GN_RCL_SMD:C0402(1005M), symbol 001_Basic_PassiveComponents:101_Capacitor
- removed R? (x2): 100k, 001_GN_RCL_SMD:R0402(1005M), symbol 001_Basic_PassiveComponents:001_Resistor
- removed R?: 10k, 001_GN_RCL_SMD:R0402(1005M), symbol 001_Basic_PassiveComponents:001_Resistor
- added C?: 10pF, 001_GN_RCL_SMD:C0201(0603M), symbol 001_Basic_PassiveComponents:101_Capacitor
- added C? (x8): 100nF, 001_GN_RCL_SMD:C0201(0603M), symbol 001_Basic_PassiveComponents:101_Capacitor
- added C? (x4): 4.7uF, 001_GN_RCL_SMD:C0402(1005M), symbol 001_Basic_PassiveComponents:101_Capacitor
- added D?: XL-1010SURUBC, 003_GN_SMALL-SEMI_SMD:LED-4_1010, symbol 004_Basic_Co-PackagedSemiconductor:XL-1010SURUBC
- added FB?: 120R, 001_GN_RCL_SMD:L0603(1608M), symbol 001_Basic_PassiveComponents:301_FerriteBead
- added J?: Conn_01x05, symbol 302_Link_W2B-Connector:Conn_01x05
- added L?: 4.7uH, 008_GN_POWER-CHOKE_SMD:MC-0530, symbol 001_Basic_PassiveComponents:202_PowerChoke
- added NT? (x4): NetCNVT-2, symbol 300_Link_NetCNVT:NetCNVT-2
- added R?: 68k, 001_GN_RCL_SMD:R0201(0603M), symbol 001_Basic_PassiveComponents:001_Resistor
- added R? (x6): 10k, 001_GN_RCL_SMD:R0201(0603M), symbol 001_Basic_PassiveComponents:001_Resistor
- added R? (x2): 1k, 001_GN_RCL_SMD:R0201(0603M), symbol 001_Basic_PassiveComponents:001_Resistor
- added R?: 21.5k, 001_GN_RCL_SMD:R0201(0603M), symbol 001_Basic_PassiveComponents:001_Resistor
- added R?: 100k, 001_GN_RCL_SMD:R0201(0603M), symbol 001_Basic_PassiveComponents:001_Resistor
- added U?: JW5393FSOTI, 003_GN_SMALL-SEMI_SMD:SOT-563, symbol 204_Power_SMPS-Convertor:JW5393FSOTI
- added U?: ZD25Q80BNIGR, 003_GN_SMALL-SEMI_SMD:DFN-8_1515, symbol 108_IntegratedCircuit_Storage:ZD25Q80BNIGR
- C? (x2): footprint 001_GN_RCL_SMD:C0402(1005M) -> 001_GN_RCL_SMD:C0201(0603M)
- R? (x2): footprint 001_GN_RCL_SMD:R0402(1005M) -> 001_GN_RCL_SMD:R0201(0603M)
Connections:
- net +3V3: now also C?.1, C?.1, C?.1, C?.1, FB?.1, R?.2, U?.8 (Vin)
- net BOOT0: now also R?.1
- net DAP_CLK: now also NT?.2
- net DAP_DIO: now also NT?.2
- net DAP_Rx: now also NT?.1
- net DAP_Tx: now also NT?.1
- net FL_SCK: now also U?.6 (CLK)
- net FL_~{CS}: now also R?.1, U?.1 (~{CS})
- net GND: now also C?.1, C?.2, C?.2, C?.2, C?.2, C?.2, C?.2, C?.2, C?.2, C?.2, C?.2, C?.2, D?.1 (Cathode), D?.4 (Cathode), R?.2, R?.2, R?.2, R?.2, U?.3 (GND), U?.4 (GND), U?.EP
- net LED_B: now also R?.2
- net LED_R: now also R?.2
- net SWO_TDO: now also J?.5, NT?.2
- net SWRST_SRST: now also J?.4
- net TDI: now also J?.1
- net TRST: now also NT?.2
- net UART-CC1: now also R?.2
- net UART-CC2: now also R?.1
- net VBUS: now also C?.1, C?.1, R?.2, U?.1 (VIN)
- net VDC: now also R?.1, R?.2
- net ~{RST}: now also C?.1
- net at U?.10 (V_1V8): now also C?.1
- net at U?.11 (XTAL_OUT), X?.3: now also C?.2
- net at U?.9 (V_3V3): now also C?.1
- net SWCLK renamed SWCLK_TCK
- net SWCLK_TCK: now also J?.3
- net SWDIO renamed SWDIO_TMS
- net SWDIO_TMS: now also J?.2
- new net: R?.1, R?.1, U?.6 (FB)
- new net: R?.1, U?.7 (~{HLD})
- new net: D?.2 (Anode), R?.1
- new net: D?.3 (Anode), R?.1
- new net: C?.2, L?.1, U?.2 (SW)
- new net: C?.1, U?.4 (BST)
- new net: R?.1, U?.5 (EN)
- new net: R?.1, U?.3 (~{WP})
- new net +3.3VP: C?.1, C?.1, FB?.2, L?.2, R?.2
- new net FL_MISO: NT?.1, U?.2 (DO)
- new net FL_MOSI: NT?.1, U?.5 (DI)
- no-connect marks 14 -> 12
Other:
- moved on the sheet: C?, J?, R?, U?, U?A, U?B, U?C, X?

Commit message: Update DAPlink_CC.kicad_sch
Parts:
- added C? (x2): 100nF, 001_GN_RCL_SMD:C0201(0603M), symbol 001_Basic_PassiveComponents:101_Capacitor
- added U? (x2): HC32L110B6YA, 104_SP_SMALL_SMD:CSP-16_1614, symbol 107_IntegratedCircuit_MicroController:HC32L110B6YA
Connections:
- net +3V3: now also U?.C4 (Vin)
- net GND: now also C?.2, C?.2, U?.B4 (GND)
- new net: C?.1, U?.B2 (~{RST})
- new net: C?.1, U?.C3 (Vcap)
Other:
- moved on the sheet: R?, U?A

Commit message: Update DAPlink_CC.kicad_sch
Parts:
- removed J?: Conn_01x05, symbol 302_Link_W2B-Connector:Conn_01x05
- added C? (x4): 100nF, 001_GN_RCL_SMD:C0201(0603M), symbol 001_Basic_PassiveComponents:101_Capacitor
- added D? (x7): LESD11LL5.0CT5G, 002_GN_TWO-PIN_PLASTIC_SMD:SOD-123, symbol 002_Basic_SingleSemiconductor:007_Diode_ESD_Bi
- added R? (x5): 10k, 001_GN_RCL_SMD:R0201(0603M), symbol 001_Basic_PassiveComponents:001_Resistor
- added U? (x3): LP5240HVF, 104_SP_SMALL_SMD:CSP-4_S7575, symbol 110_IntegratedCircuit_Interface:LP5240HVF
- added U? (x3): DIO32220LP10, 003_GN_SMALL-SEMI_SMD:QFN-10_1814, symbol 110_IntegratedCircuit_Interface:DIO32220LP10
- C?: value 100nF -> 4.7uF
- R?: value 5.1k -> 10k
- R? (x2): value 10k -> 100k
Connections:
- net +3.3VP: now also U?.A2 (Vin)
- net +3V3: now also R?.1, R?.2, C?.1, C?.1, C?.1, C?.1, R?.1, U?.9 (Vin), U?.9 (Vin), U?.9 (Vin)
- net DAP_CLK: now also D?.2 (Anode)
- net DAP_DIO: now also D?.2 (Anode)
- net DAP_Rx: now also D?.2 (Anode)
- net DAP_Tx: now also D?.2 (Anode)
- net DN: now also D?.1 (Cathode)
- net DP: now also D?.1 (Cathode)
- net GND: now also C?.2, C?.2, C?.2, C?.2, D?.1 (Cathode), D?.1 (Cathode), D?.1 (Cathode), D?.1 (Cathode), D?.2 (Anode), D?.2 (Anode), D?.2 (Anode), R?.2, R?.2, U?.4 (GND), U?.4 (GND), U?.4 (GND), U?.B1 (GND), U?.B1 (GND), U?.B1 (GND)
- net SWCLK_TCK: now also U?.2 (NO1), U?.7 (NC2)
- net SWD-SBU1: now also U?.3 (COM1)
- net SWD-SBU2: now also U?.5 (COM2)
- net SWDIO_TMS: now also U?.1 (NC1), U?.6 (NO2)
- net SWO_TDO: now also U?.6 (NO2)
- net TDI: now also U?.2 (NO1)
- net UART-CC1: now also U?.B3 (P01), U?.3 (COM1)
- net UART-CC2: now also U?.A4 (P02), U?.5 (COM2)
- net UART-Rx: now also U?.2 (NO1), U?.7 (NC2), U?.7 (NC2); no longer J?.A11 (Rx2_P), J?.B11 (Rx1_P)
- net UART-Tx: now also U?.1 (NC1), U?.1 (NC1), U?.6 (NO2); no longer J?.A10 (Rx2_N), J?.B10 (Rx1_N)
- net VBUS: now also D?.1 (Cathode), U?.A2 (Vin)
- net VDC: now also R?.1, U?.A2 (Vin); no longer R?.1, R?.2
- net Isns_N: now reaches U?.A1 (P26)
- net Isns_N: now also R?.1, R?.2
- net 3V3_SEL: now reaches U?.A2 (P35)
- net 3V3_SEL: now also U?.B2 (EN)
- net 5V_SEL: now reaches U?.A3 (P36)
- net 5V_SEL: now also U?.B2 (EN)
- net JTAG_SEL: now reaches U?.B1 (P25)
- net JTAG_SEL: now also U?.10 (SEL)
- net Isns_P: now reaches U?.C1 (P24)
- net Isns_P: now also R?.1, R?.2
- net DIR_SEL: now reaches U?.C2 (P23)
- net DIR_SEL: now also U?.10 (SEL), U?.10 (SEL)
- net VOE: now reaches U?.D1 (P14)
- net VOE: now also U?.B2 (EN)
- net ~{OE}: now reaches U?.D2 (P15)
- net ~{OE}: now also R?.2, U?.8 (~{OE}), U?.8 (~{OE}), U?.8 (~{OE})
- net AUX_SWDIO: now reaches U?.D3 (P27)
- net AUX_SWCLK: now reaches U?.D4 (P31)
- new net DBG-RxN: J?.A10 (Rx2_N), J?.B10 (Rx1_N), U?.3 (COM1)
- new net DBG-RxP: J?.A11 (Rx2_P), J?.B11 (Rx1_P), U?.5 (COM2)
- new net VDD: R?.1, U?.A1 (Vout), U?.A1 (Vout), U?.A1 (Vout)
- no-connect marks 12 -> 8
Other:
- moved on the sheet: C?, D?, NT?, R?, U?, U?A, U?B, U?C, X?

Commit message: Update schematics
Parts:
- removed C? (x3): 100nF, 001_GN_RCL_SMD:C0201(0603M), symbol 001_Basic_PassiveComponents:101_Capacitor
- removed D? (x7): LESD11LL5.0CT5G, 002_GN_TWO-PIN_PLASTIC_SMD:SOD-123, symbol 002_Basic_SingleSemiconductor:007_Diode_ESD_Bi
- removed J? (x2): USB_TypeC-24, symbol 306_Link_USB-Connector:USB_TypeC-24
- removed R?: 10k, 001_GN_RCL_SMD:R0201(0603M), symbol 001_Basic_PassiveComponents:001_Resistor
- removed R? (x2): 100k, 001_GN_RCL_SMD:R0201(0603M), symbol 001_Basic_PassiveComponents:001_Resistor
- removed U? (x3): LP5240HVF, 104_SP_SMALL_SMD:CSP-4_S7575, symbol 110_IntegratedCircuit_Interface:LP5240HVF
- removed U? (x3): DIO32220LP10, 003_GN_SMALL-SEMI_SMD:QFN-10_1814, symbol 110_IntegratedCircuit_Interface:DIO32220LP10
- added C? (x3): 100nF, 001_GN_RCL_SMD:C0201(0603M), symbol 001_Basic_PassiveComponents:101_Capacitor
- added U? (x3): LP5240HVF, 104_SP_SMALL_SMD:CSP-4_S7575, symbol 110_IntegratedCircuit_Interface:LP5240HVF
- added U? (x3): DIO32220LP10, 003_GN_SMALL-SEMI_SMD:QFN-10_1814, symbol 110_IntegratedCircuit_Interface:DIO32220LP10
Connections:
- net +3.3VP: now also U?.A2 (Vin)
- net +3V3: now also C?.1, C?.1, C?.1, U?.9 (Vin), U?.9 (Vin), U?.9 (Vin)
- net 3V3_SEL: now also U?.B2 (EN)
- net 5V_SEL: now also U?.B2 (EN)
- net DBG-RxN: now also U?.3 (COM1)
- net DBG-RxP: now also U?.5 (COM2)
- net DIR_SEL: now also U?.10 (SEL), U?.10 (SEL)
- net GND: now also C?.2, C?.2, C?.2, U?.4 (GND), U?.4 (GND), U?.4 (GND), U?.B1 (GND), U?.B1 (GND), U?.B1 (GND)
- net JTAG_SEL: now also U?.10 (SEL)
- net SWCLK_TCK: now also U?.2 (NO1), U?.7 (NC2)
- net SWD-SBU1: now also U?.3 (COM1)
- net SWD-SBU2: now also U?.5 (COM2)
- net SWDIO_TMS: now also U?.1 (NC1), U?.6 (NO2)
- net SWO_TDO: now also U?.6 (NO2)
- net TDI: now also U?.2 (NO1)
- net UART-CC1: now also U?.3 (COM1)
- net UART-CC2: now also U?.5 (COM2)
- net UART-Rx: now also U?.2 (NO1), U?.7 (NC2), U?.7 (NC2)
- net UART-Tx: now also U?.1 (NC1), U?.1 (NC1), U?.6 (NO2)
- net VBUS: now also U?.A2 (Vin)
- net VDC: now also U?.A2 (Vin)
- net VDD: now also U?.A1 (Vout), U?.A1 (Vout), U?.A1 (Vout)
- net VOE: now also U?.B2 (EN)
- net ~{OE}: now also U?.8 (~{OE}), U?.8 (~{OE}), U?.8 (~{OE})
Other:
- added sheet CONN (CONN.kicad_sch)
- moved on the sheet: C?, D?, FB?, NT?, R?, U?, U?A, U?B, U?C, X?

Commit message: Complete schematics
Nightly update
Parts:
- removed NT? (x3): NetCNVT-2, symbol 300_Link_NetCNVT:NetCNVT-2
- removed U?: LP5240HVF, 104_SP_SMALL_SMD:CSP-4_S7575, symbol 110_IntegratedCircuit_Interface:LP5240HVF
- added C13, C15, C18: 100nF, 001_GN_RCL_SMD:C0201(0603M), symbol 001_Basic_PassiveComponents:101_Capacitor
- added NT2, NT3, NT4: NetCNVT-2, 301_MECH_DRAWING:NetCNVT, symbol 300_Link_NetCNVT:NetCNVT-2
- added R16: 10k, 001_GN_RCL_SMD:R0201(0603M), symbol 001_Basic_PassiveComponents:001_Resistor
- L1: renamed from L?; footprint 008_GN_POWER-CHOKE_SMD:MC-0530 -> 008_GN_POWER-CHOKE_SMD:MC-2520
- NT1: renamed from NT?; footprint (none) -> 301_MECH_DRAWING:NetCNVT
- gave numbers to parts that had none: 49
Connections:
- net +3.3VP: now also C13.1
- net DAP_DIO: now also NT2.2
- net DAP_Rx: now also NT4.1
- net DAP_Tx: now also NT3.1
- net FL_MISO: now also NT2.1
- net GND: now also C13.2, C15.2, C18.2, R16.1
- net JTAG_SEL: now also R16.2
- net SWO_TDO: now also NT4.2
- net TRST: now also NT3.2
- net VBUS: now also C15.1; no longer C10.1, C5.1, C9.1, R10.2, U2.7 (Vin_5V), U5.1 (VIN), U7.A2 (Vin)
- net VDD: now also C18.1
- net VOE renamed IDL-D
- new net +5VP: C10.1, C5.1, C9.1, R10.2, U2.7 (Vin_5V), U5.1 (VIN), U7.A2 (Vin)
Other:
- sheet CONN ports: added AUX_SWCLK, AUX_SWDIO, DAP_CLK, DAP_DIO, DAP_Rx, DAP_Tx, DBG-RxN, DBG-RxP, DN, DP, DVC-DN, DVC-DP, IDL-D, KEY, SWCLK_TCK, SWD-SBU1, SWD-SBU2, SWDIO_TMS, SWRST_SRST, TRST, UART-CC1, UART-CC2; removed none
- moved on the sheet: C17, C22, C23, R15, U10, U6A, U9
