File: DAPlink_CC.kicad_sch (KiCad schematic)
At the start: 58 parts, among them U1 ZD25Q80BNIGR, U10 DIO32220LP10, U2 SL2.1S, U3 GD32F350G8U6, U4 LP5240HVF, U5 JW5393FSOTI, U6 HC32L110B6YA, U7 LP5240HVF, U8 DIO32220LP10, U9 DIO32220LP10, X1 002_Xtal-4

Commit message: Update DAPlink_CC.kicad_sch
Connections:
- net 3V3_SEL: now also U6.B1 (P25); no longer U6.A2 (P35)
- net 5V_SEL: now also U6.A1 (P26); no longer U6.A3 (P36)
- net Isns_N: now also U6.A3 (P36); no longer U6.A1 (P26)
- net Isns_P: now also U6.A2 (P35); no longer U6.C1 (P24)
- net JTAG_SEL: now also U6.C1 (P24); no longer U6.B1 (P25)
Other:
- moved on the sheet: R8, R9
Changed lines of the file:
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@@
 (kicad_sch (version 20211123) (generator eeschema)
   (paper "A4")
+  (junction (at 91.44 101.6) (diameter 0) (color 0 0 0 0)
+  )
   (junction (at 38.1 83.82) (diameter 0) (color 0 0 0 0)
   )
@@
   (junction (at 157.48 175.26) (diameter 0) (color 0 0 0 0)
   )
-  (junction (at 93.98 101.6) (diameter 0) (color 0 0 0 0)
-  )
   (junction (at 162.56 160.02) (diameter 0) (color 0 0 0 0)
   )
@@
     (stroke (width 0) (type default) (color 0 0 0 0))
   )
-  (wire (pts (xy 99.06 114.3) (xy 114.3 114.3))
+  (wire (pts (xy 104.14 114.3) (xy 114.3 114.3))
     (stroke (width 0) (type default) (color 0 0 0 0))
   )
@@
     (stroke (width 0) (type default) (color 0 0 0 0))
   )
-  (wire (pts (xy 93.98 78.74) (xy 93.98 81.28))
+  (wire (pts (xy 91.44 78.74) (xy 91.44 81.28))
     (stroke (width 0) (type default) (color 0 0 0 0))
   )
@@
     (stroke (width 0) (type default) (color 0 0 0 0))
   )
-  (wire (pts (xy 93.98 91.44) (xy 93.98 101.6))
+  (wire (pts (xy 91.44 91.44) (xy 91.44 101.6))
     (stroke (width 0) (type default) (color 0 0 0 0))
   )
@@
     (stroke (width 0) (type default) (color 0 0 0 0))
   )
-  (wire (pts (xy 101.6 104.14) (xy 114.3 104.14))
+  (wire (pts (xy 104.14 104.14) (xy 114.3 104.14))
     (stroke (width 0) (type default) (color 0 0 0 0))
   )
@@
     (stroke (width 0) (type default) (color 0 0 0 0))
   )
-  (wire (pts (xy 93.98 114.3) (xy 93.98 116.84))
+  (wire (pts (xy 91.44 114.3) (xy 91.44 116.84))
     (stroke (width 0) (type default) (color 0 0 0 0))
   )
@@
     (stroke (width 0.508) (type default) (color 0 0 0 0))
   )
-  (wire (pts (xy 93.98 101.6) (xy 93.98 104.14))
-    (stroke (width 0) (type default) (color 0 0 0 0))
-  )
   (wire (pts (xy 218.44 142.24) (xy 218.44 144.78))
     (stroke (width 0) (type default) (color 0 0 0 0))
@@
     (stroke (width 0) (type default) (color 0 0 0 0))
   )
-  (wire (pts (xy 101.6 96.52) (xy 101.6 104.14))
-    (stroke (width 0) (type default) (color 0 0 0 0))
-  )
   (wire (pts (xy 66.04 187.96) (xy 68.58 187.96))
     (stroke (width 0) (type default) (color 0 0 0 0))
@@
     (stroke (width 0) (type default) (color 0 0 0 0))
   )
+  (wire (pts (xy 91.44 101.6) (xy 91.44 104.14))
+    (stroke (width 0) (type default) (color 0 0 0 0))
+  )
   (wire (pts (xy 50.8 187.96) (xy 55.88 187.96))
     (stroke (width 0) (type default) (color 0 0 0 0))
@@
     (stroke (width 0) (type default) (color 0 0 0 0))
   )
-  (wire (pts (xy 99.06 101.6) (xy 93.98 101.6))
+  (wire (pts (xy 91.44 101.6) (xy 99.06 101.6))
     (stroke (width 0) (type default) (color 0 0 0 0))
   )
@@
     (stroke (width 0) (type default) (color 0 0 0 0))
   )
-  (wire (pts (xy 101.6 96.52) (xy 86.36 96.52))
-    (stroke (width 0) (type default) (color 0 0 0 0))
-  )
-  (wire (pts (xy 99.06 114.3) (xy 99.06 101.6))
+  (wire (pts (xy 99.06 96.52) (xy 86.36 96.52))
     (stroke (width 0) (type default) (color 0 0 0 0))
   )
@@
     (effects (font (size 1.27 1.27)) (justify right bottom))
   )
-  (label "Isns_N" (at 104.14 114.3 0)
-    (effects (font (size 1.27 1.27)) (justify left bottom))
-  )
-  (label "5V_SEL" (at 157.48 114.3 180)
+  (label "Isns_N" (at 157.48 114.3 180)
     (effects (font (size 1.27 1.27)) (justify right bottom))
   )
+  (label "5V_SEL" (at 104.14 114.3 0)
+    (effects (font (size 1.27 1.27)) (justify left bottom))
+  )
   (label "TRST" (at 274.32 25.4 180)
     (effects (font (size 1.27 1.27)) (justify right bottom))
@@
     (effects (font (size 1.27 1.27)) (justify right bottom))
   )
+  (label "Isns_P" (at 99.06 96.52 180)
+    (effects (font (size 1.27 1.27)) (justify right bottom))
+  )
   (label "UART-CC2" (at 226.06 149.86 180)
     (effects (font (size 1.27 1.27)) (justify right bottom))
@@
     (effects (font (size 1.27 1.27)) (justify left bottom))
   )
-  (label "Isns_P" (at 104.14 104.14 0)
-    (effects (font (size 1.27 1.27)) (justify left bottom))
+  (label "Isns_P" (at 157.48 109.22 180)
+    (effects (font (size 1.27 1.27)) (justify right bottom))
   )
   (label "DP" (at 231.14 101.6 0)
@@
     (effects (font (size 1.27 1.27)) (justify right bottom))
   )
+  (label "Isns_N" (at 99.06 101.6 180)
+    (effects (font (size 1.27 1.27)) (justify right bottom))
+  )
   (label "UART-CC1" (at 104.14 88.9 0)
     (effects (font (size 1.27 1.27)) (justify left bottom))
@@
     (effects (font (size 1.27 1.27)) (justify left bottom))
   )
-  (label "3V3_SEL" (at 157.48 109.22 180)
-    (effects (font (size 1.27 1.27)) (justify right bottom))
+  (label "3V3_SEL" (at 104.14 109.22 0)
+    (effects (font (size 1.27 1.27)) (justify left bottom))
   )
   (label "KEY" (at 231.14 93.98 0)
@@
     (effects (font (size 1.27 1.27)) (justify right bottom))
   )
-  (label "JTAG_SEL" (at 104.14 109.22 0)
+  (label "JTAG_SEL" (at 104.14 104.14 0)
     (effects (font (size 1.27 1.27)) (justify left bottom))
   )
@@
     (pin "2")
   )
-  (symbol (lib_id "001_Basic_PassiveComponents:001_Resistor") (at 93.98 109.22 270) (unit 1)
+  (symbol (lib_id "001_Basic_PassiveComponents:001_Resistor") (at 91.44 109.22 270) (unit 1)
     (in_bom yes) (on_board yes)
-    (property "Reference" "R9" (id 0) (at 93.98 104.14 90)
+    (property "Reference" "R9" (id 0) (at 91.44 104.14 90)
       (effects (font (size 1.27 1.27)) (justify left))
     )
-    (property "Value" "10k" (id 1) (at 93.98 114.3 90)
+    (property "Value" "10k" (id 1) (at 91.44 114.3 90)
       (effects (font (size 1.27 1.27)) (justify left))
     )
-    (property "Footprint" "001_GN_RCL_SMD:R0201(0603M)" (id 2) (at 99.06 109.22 0)
+    (property "Footprint" "001_GN_RCL_SMD:R0201(0603M)" (id 2) (at 96.52 109.22 0)
       (effects (font (size 1.27 1.27)) hide)
     )
-    (property "Datasheet" "" (id 3) (at 97.79 105.41 0)
+    (property "Datasheet" "" (id 3) (at 95.25 105.41 0)
       (effects (font (size 1.27 1.27)) hide)
     )
-    (property "Symbol type" "Alternate Source" (id 4) (at 101.6 109.22 0)
+    (property "Symbol type" "Alternate Source" (id 4) (at 99.06 109.22 0)
       (effects (font (size 1.27 1.27)) hide)
     )
@@
     (pin "1")
   )
-  (symbol (lib_id "001_Basic_PassiveComponents:001_Resistor") (at 93.98 86.36 270) (unit 1)
+  (symbol (lib_id "001_Basic_PassiveComponents:001_Resistor") (at 91.44 86.36 270) (unit 1)
     (in_bom yes) (on_board yes)
-    (property "Reference" "R8" (id 0) (at 93.98 81.28 90)
+    (property "Reference" "R8" (id 0) (at 91.44 81.28 90)
       (effects (font (size 1.27 1.27)) (justify left))
     )
-    (property "Value" "10k" (id 1) (at 93.98 91.44 90)
+    (property "Value" "10k" (id 1) (at 91.44 91.44 90)
       (effects (font (size 1.27 1.27)) (justify left))
     )
-    (property "Footprint" "001_GN_RCL_SMD:R0201(0603M)" (id 2) (at 99.06 86.36 0)
+    (property "Footprint" "001_GN_RCL_SMD:R0201(0603M)" (id 2) (at 96.52 86.36 0)
       (effects (font (size 1.27 1.27)) hide)
     )
-    (property "Datasheet" "" (id 3) (at 97.79 82.55 0)
+    (property "Datasheet" "" (id 3) (at 95.25 82.55 0)
       (effects (font (size 1.27 1.27)) hide)
     )
-    (property "Symbol type" "Alternate Source" (id 4) (at 101.6 86.36 0)
+    (property "Symbol type" "Alternate Source" (id 4) (at 99.06 86.36 0)
       (effects (font (size 1.27 1.27)) hide)
     )
@@
     (pin "2")
   )
-  (symbol (lib_id "PowerPort:VDC") (at 93.98 78.74 0) (unit 1)
+  (symbol (lib_id "PowerPort:VDC") (at 91.44 78.74 0) (unit 1)
     (in_bom yes) (on_board yes) (fields_autoplaced)
-    (property "Reference" "#PWR028" (id 0) (at 93.98 81.28 0)
+    (property "Reference" "#PWR028" (id 0) (at 91.44 81.28 0)
       (effects (font (size 1.27 1.27)) hide)
     )
-    (property "Value" "VDC" (id 1) (at 93.98 73.66 0))
-    (property "Footprint" "" (id 2) (at 93.98 78.74 0)
+    (property "Value" "VDC" (id 1) (at 91.44 73.66 0))
+    (property "Footprint" "" (id 2) (at 91.44 78.74 0)
       (effects (font (size 1.27 1.27)) hide)
     )
-    (property "Datasheet" "" (id 3) (at 93.98 78.74 0)
+    (property "Datasheet" "" (id 3) (at 91.44 78.74 0)
       (effects (font (size 1.27 1.27)) hide)
     )
@@
     (pin "2")
   )
-  (symbol (lib_id "PowerPort:GND") (at 93.98 116.84 0) (mirror y) (unit 1)
+  (symbol (lib_id "PowerPort:GND") (at 91.44 116.84 0) (mirror y) (unit 1)
     (in_bom yes) (on_board yes) (fields_autoplaced)
-    (property "Reference" "#PWR029" (id 0) (at 93.98 123.19 0)
+    (property "Reference" "#PWR029" (id 0) (at 91.44 123.19 0)
       (effects (font (size 1.27 1.27)) hide)
     )
-    (property "Value" "GND" (id 1) (at 93.98 121.92 0))
-    (property "Footprint" "" (id 2) (at 93.98 116.84 0)
+    (property "Value" "GND" (id 1) (at 91.44 121.92 0))
+    (property "Footprint" "" (id 2) (at 91.44 116.84 0)
       (effects (font (size 1.27 1.27)) hide)
     )
-    (property "Datasheet" "" (id 3) (at 93.98 116.84 0)
+    (property "Datasheet" "" (id 3) (at 91.44 116.84 0)
       (effects (font (size 1.27 1.27)) hide)
     )
@@
     (pin "C3")
     (pin "C4")
-    (pin "A1" (alternate "ADC_IN1"))
-    (pin "A2")
-    (pin "A3")
+    (pin "A1")
+    (pin "A2" (alternate "ADC_IN5"))
+    (pin "A3" (alternate "ADC_IN6"))
     (pin "A4" (alternate "ADC_IN8"))
     (pin "B1")
     (pin "B3" (alternate "ADC_IN7"))
-    (pin "C1" (alternate "ADC_IN0"))
+    (pin "C1")
     (pin "C2")
     (pin "D1")
@@
     (pin "C4")
     (pin "A1")
-    (pin "A2")
-    (pin "A3")
-    (pin "A4")
+    (pin "A2" (alternate "ADC_IN5"))
+    (pin "A3" (alternate "ADC_IN6"))
+    (pin "A4" (alternate "ADC_IN8"))
     (pin "B1")
-    (pin "B3")
+    (pin "B3" (alternate "ADC_IN7"))
     (pin "C1")
     (pin "C2")
     (pin "D1")
     (pin "D2")
-    (pin "D3")
-    (pin "D4")
+    (pin "D3" (alternate "SWDIO"))
+    (pin "D4" (alternate "SWCLK"))
   )
   (symbol (lib_id "PowerPort:+3V3") (at 218.44 142.24 0) (unit 1)
