File: DAPlink_CC.kicad_pcb (KiCad board)
At the start: 6 copper layers, 5.9 x 12 mm, 89 parts, among them J1 USB_TypeC-24, J2 Conn_01x04, J3 USB_TypeC-24, J4 Conn_01x02, J5 Conn_01x02, J6 Conn_01x04, Q1 YJL2101W, Q2 TPM7002DFN3, U1 ZD25Q80BNIGR, U10 DIO32220LP10, U11 AW33901FCR, U2 SL2.1S, U3 GD32F350G8U6, U4 LP5240HVF, U5 JW5393FSOTI, U6 HC32L110B6YA, U7 LP5240HVF, U8 DIO32220LP10, U9 DIO32220LP10, X1 12MHz

Commit message: Update layout
Nightly update
Parts:
- R18, R20: footprint 001_GN_RCL_SMD:R0201(0603M) -> 001_GN_RCL_SMD:R0402(1005M); moved to B.Cu
- moved D1 46.1 mm to (116.8, 97.2)
- moved R2 42.1 mm to (112.0, 97.1), turned to 180 degrees
- moved R16 40.7 mm to (112.5, 103.1)
- moved R1 38.4 mm to (112.0, 96.5), turned to 180 degrees
- moved U3 20.1 mm to (110.1, 97.1)
- moved J1 20.0 mm to (95.0, 100.0)
- moved R18 17.0 mm to (113.1, 98.0), turned to -90 degrees
- moved X1 15.4 mm to (103.5, 102.0), turned to 90 degrees
- moved U1 15.3 mm to (106.5, 102.5)
- moved U6 14.3 mm to (110.0, 102.6), turned to -90 degrees
- moved R20 13.4 mm to (113.1, 102.0), turned to 90 degrees
- moved U2 10.3 mm to (103.8, 97.5), turned to -90 degrees
- moved U11 5.15 mm to (106.2, 107.5)
- moved D9 1.01 mm to (116.2, 98.4), turned to 0 degrees
Connections:
- U10 pad 1: /SWDIO_TMS -> /SWCLK_TCK
- U10 pad 2: /SWCLK_TCK -> /SWDIO_TMS
- U10 pad 6: /SWDIO_TMS -> /SWCLK_TCK
- U10 pad 7: /SWCLK_TCK -> /SWDIO_TMS
- U8 pad 1: /UART-Rx -> /UART-Tx
- U8 pad 2: /TDI -> /SWO_TDO
- U8 pad 3: /DBG-RxP -> /DBG-RxN
- U8 pad 5: /DBG-RxN -> /DBG-RxP
- U8 pad 6: /SWO_TDO -> /TDI
- U8 pad 7: /UART-Tx -> /UART-Rx
Routing:
- net /DBG-RxN: track 5.17 -> 11.2 mm, vias 2 -> 3
- net /SWD-SBU1: track 1.31 -> 7.04 mm, vias 1 -> 2
- net /UART-CC2: track 3.75 -> 9.40 mm, vias 2 -> 3
- net /UART-CC1: track 1.31 -> 6.73 mm, vias 1 -> 2
- net /UART-Tx: track 0.00 -> 4.68 mm, vias 0 -> 3
- net /DBG-RxP: track 7.53 -> 11.6 mm, vias 2 -> 3
- net /SWD-SBU2: track 3.22 -> 6.57 mm, vias 2 -> 3
- net /UART-Rx: track 0.00 -> 3.18 mm
- net Net-(D1-Pad3): track 0.00 -> 2.07 mm
- net +3.3VP: track 0.00 -> 1.43 mm, vias 0 -> 1
- net /5V_SEL: track 0.00 -> 1.34 mm
- net /SWCLK_TCK: track 4.86 -> 6.13 mm, vias 2 -> 3
- net /TDI: track 0.00 -> 0.97 mm, vias 0 -> 1
- net /3V3_SEL: track 0.00 -> 0.95 mm, vias 0 -> 1
- net +3V3: track 0.00 -> 0.57 mm, vias 0 -> 3
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- added copper zone on F.Cu, net /JTAG_SEL
- added copper zone on F.Cu, net GND
Other:
- board size 5.9 x 12 mm -> 34 x 12.5 mm

Commit message: Nightly update
Parts:
- C13, C15, C18: footprint 001_GN_RCL_SMD:C0201(0603M) -> 001_GN_RCL_SMD:C0402(1005M)
- NT3, NT4: moved to B.Cu
- moved C17 41.8 mm to (110.4, 101.2), turned to -90 degrees
- moved C20 41.6 mm to (112.4, 102.5), turned to 180 degrees
- moved C13 41.2 mm to (111.8, 105.3)
- moved C21 39.7 mm to (112.4, 100.0), turned to 180 degrees
- moved C11 39.6 mm to (111.8, 97.0), turned to 180 degrees
- moved C6 39.4 mm to (111.8, 98.2), turned to 180 degrees
- moved C23 39.1 mm to (109.2, 101.2), turned to -90 degrees
- moved C22 38.4 mm to (111.0, 101.2), turned to -90 degrees
- moved NT3 37.5 mm to (111.8, 99.8)
- moved NT4 36.2 mm to (111.8, 100.0)
- moved C24 35.2 mm to (112.6, 98.4), turned to -90 degrees
- moved R11 35.1 mm to (111.8, 96.4), turned to 180 degrees
- moved R12 33.9 mm to (111.8, 97.6)
- moved C8 32.9 mm to (108.2, 98.2)
- moved C15 26.5 mm to (100.5, 97.4)
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Connections:
- C15 pad 1: VBUS -> +5VP
Routing:
- net Net-(D1-Pad2): track 0.00 -> 2.99 mm
- net Net-(D1-Pad3): track 2.07 -> 3.29 mm
Other:
- outline, holes or cut-outs redrawn

Commit message: Daily update
Parts:
- C13, C15, C18, C9, NT1, NT2: moved to B.Cu
- NT4, X1: moved to F.Cu
- moved C18 43.0 mm to (116.8, 103.1)
- moved R15 40.0 mm to (112.0, 101.6), turned to 90 degrees
- moved R6 39.8 mm to (108.5, 102.8), turned to 180 degrees
- moved R4 39.4 mm to (106.4, 100.5)
- moved R7 39.3 mm to (108.5, 103.4)
- moved R3 39.0 mm to (106.6, 98.4), turned to -90 degrees
- moved C1 37.1 mm to (105.5, 100.8), turned to -90 degrees
- moved C5 35.9 mm to (104.0, 104.9), turned to 180 degrees
- moved R9 35.5 mm to (108.2, 101.2), turned to 90 degrees
- moved C3 34.7 mm to (103.6, 100.8), turned to 90 degrees
- moved FB1 34.6 mm to (103.4, 96.6), turned to 180 degrees
- moved R8 34.5 mm to (108.5, 102.1), turned to 180 degrees
- moved C2 34.1 mm to (106.4, 99.9)
- moved C4 33.3 mm to (104.2, 100.8), turned to 90 degrees
- moved C10 32.7 mm to (102.6, 100.1), turned to -90 degrees
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Connections:
- U6 pad 16: (no net) -> unconnected-(U6-Pad16)
- U6 pad 17: (no net) -> unconnected-(U6-Pad17)
- U6 pad 18: (no net) -> unconnected-(U6-Pad18)
- U6 pad 7: (no net) -> unconnected-(U6-Pad7)
- U6 pad EP: (no net) -> GND
Routing:
- net /SWDIO_TMS: track 6.92 -> 24.8 mm
- net /DVC-DP: track 2.39 -> 20.2 mm
- net VDC: track 11.3 -> 28.8 mm, vias 5 -> 6
- net /DVC-DN: track 4.60 -> 19.7 mm, vias 2 -> 3
- net VDD: track 1.71 -> 16.2 mm, vias 2 -> 3
- net /3V3_SEL: track 0.95 -> 12.8 mm, vias 1 -> 2
- net /SWCLK_TCK: track 6.13 -> 17.1 mm
- net /DIR_SEL: track 0.00 -> 10.8 mm, vias 0 -> 2
- net /SWO_TDO: track 0.00 -> 10.4 mm, vias 0 -> 1
- net /~{OE}: track 0.00 -> 9.28 mm, vias 0 -> 3
- net /DAP_Tx: track 0.00 -> 9.20 mm, vias 0 -> 3
- net /DAP_CLK: track 0.00 -> 8.83 mm, vias 0 -> 3
- net /TRST: track 0.00 -> 8.13 mm
- net /DAP_Rx: track 0.00 -> 7.52 mm, vias 0 -> 4
- net /IDL-D: track 0.00 -> 6.96 mm, vias 1 -> 2
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- added copper zone on F.Cu, net +3V3
- added copper zone on B.Cu, net VDC
- added copper zone on B.Cu, net VDD
Other:
- board size 34 x 12.5 mm -> 33 x 12.5 mm

Commit message: Nightly update
Parts:
- moved D6 3.00 mm to (101.5, 97.9)
- moved NT3 1.94 mm to (114.6, 95.4), turned to -90 degrees
- moved C14 1.43 mm to (105.0, 96.4), turned to 0 degrees
- moved R13 1.00 mm to (105.1, 99.9), turned to 0 degrees
- moved R14 1.00 mm to (104.1, 99.9), turned to 180 degrees
- moved C23 0.40 mm to (108.9, 101.1), turned to 90 degrees
- moved NT2 0.39 mm to (106.3, 97.7), turned to 90 degrees
- moved D2 0.25 mm to (101.5, 101.6)
- moved D3 0.25 mm to (101.5, 102.6)
- moved D4 0.25 mm to (101.5, 102.1)
Routing:
- net +5VP: track 0.33 -> 52.5 mm, vias 4 -> 6
- net +3.3VP: track 2.17 -> 32.8 mm
- net +3V3: track 1.05 -> 29.9 mm, vias 6 -> 7
- net /AUX_SWDIO: track 0.00 -> 24.2 mm
- net /AUX_SWCLK: track 0.00 -> 20.4 mm
- net /DAP_Rx: track 7.52 -> 27.4 mm
- net /DAP_Tx: track 9.20 -> 27.4 mm, vias 3 -> 5
- net /DAP_DN: track 0.00 -> 15.0 mm, vias 1 -> 2
- net /DAP_CLK: track 8.83 -> 21.9 mm, vias 3 -> 5
- net /DAP_DP: track 0.00 -> 12.7 mm, vias 1 -> 2
- net /KEY: track 0.00 -> 12.6 mm
- net /TDI: track 0.97 -> 12.4 mm, vias 1 -> 2
- net /UART-Tx: track 4.68 -> 15.7 mm, vias 3 -> 4
- net /DN: track 2.37 -> 13.0 mm, vias 2 -> 3
- net /SWRST_SRST: track 0.00 -> 10.6 mm, vias 0 -> 1
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- added copper zone on B.Cu, net +3.3VP
- added copper zone on F.Cu, net +3.3VP
- added copper zone on B.Cu, net +5VP
- added copper zone on F.Cu, net +5VP
- added copper zone on F.Cu, net /FL_~{CS}
- added copper zone on B.Cu, net GND
- added copper zone on In1.Cu, net GND
- added copper zone on In2.Cu, net GND
- added copper zone on In3.Cu, net GND
- added copper zone on In4.Cu, net GND
- added copper zone on B.Cu, net Net-(C12-Pad2)
- added copper zone on F.Cu, net VBUS

Commit message: Update DAPlink_CC.kicad_pcb
Routing:
- net GND: vias 39 -> 43
